File: Mini Projet Banc Test LCD/_autosave-Mini Projet Banc Test LCD.kicad_sch (KiCad schematic)
At the start: 3 parts

Commit message: kk
Parts:
- added TP1, TP2, TP4, TP5, TP6: TestPoint, Connector_Pin:Pin_D0.7mm_L6.5mm_W1.8mm_FlatFork, symbol Connector:TestPoint
Connections:
- net at A1.4 (3V3): now also TP1.1
- net at A1.5 (+5V), LCD1.1 (VDD), RV1.1: now also TP4.1
- net at A1.7 (GND), LCD1.2 (VSS), LCD1.5 (R/W)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: now also TP2.1
- net at LCD1.15 (A): now also TP5.1
- net at LCD1.16 (K): now also TP6.1
Other:
- note added: "Banc d'essais LCD"
- moved on the sheet: A1, LCD1, RV1
